File: Hardware/M5TC-2022-U4BN.kicad_sch (KiCad schematic)
At the start: 78 parts

Commit message: Updated software to clear segments
Parts:
- A1: value (none) -> Feather 328P; footprint (none) -> Module_Feather:Adafruit_Feather
- D1, D2, D3, D4: value (none) -> LED; footprint (none) -> LED_THT:LED_D5.0mm
- H1, H2, H3, H4: value (none) -> M; footprint (none) -> MountingHole:MountingHole_5.3mm_M5_Pad_Via
- J14: value (none) -> ISP; footprint (none) -> Connector_PinSocket_2.54mm:PinSocket_2x03_P2.54mm_Vertical
- Q1, Q2, Q3: value (none) -> 2N7002; footprint (none) -> Package_TO_SOT_SMD:SOT-23
- R1, R10, R11, R12, R2, R3, R4, R9: value (none) -> 10K; footprint (none) -> Resistor_SMD:R_1206_3216Metric
- R13, R14, R15, R16, R17, R18, R19, R20, R21, R22, R23, R24, R25, R26, R27, R28, R29, R30, R31, R32, R33, R5, R6, R7, R8: value (none) -> 330; footprint (none) -> Resistor_SMD:R_1206_3216Metric
- SW1, SW2, SW3, SW4: value (none) -> SW_SPDT; footprint (none) -> 4PDT_Footprint:E-Switch-EG1218
- SW5: value (none) -> SW_Coded_SH-7050; footprint (none) -> Rotary_Hex_SOIC:Rotary_Hex_6_SOIC
- SW6: value (none) -> EG4208A; footprint (none) -> 4PDT_Footprint:E-Switch-EG4208A-0-0-MFG
- TP1: value (none) -> VCC; footprint (none) -> Custom_TestPoint:TestPoint_LoopPostPad
- TP10, TP11, TP12, TP13, TP7, TP8, TP9: value (none) -> Conn_01x01; footprint (none) -> Custom_TestPoint:TestPoint_LoopPost
- TP14: value (none) -> K1; footprint (none) -> Custom_TestPoint:TestPoint_LoopPostPad
- TP15: value (none) -> K2; footprint (none) -> Custom_TestPoint:TestPoint_LoopPostPad
- TP16: value (none) -> K3; footprint (none) -> Custom_TestPoint:TestPoint_LoopPostPad
- TP17: value (none) -> SLIDE_DATA_0; footprint (none) -> Custom_TestPoint:TestPoint_LoopPostPad
- TP18: value (none) -> SLIDE_DATA_1; footprint (none) -> Custom_TestPoint:TestPoint_LoopPostPad
- TP19: value (none) -> SLIDE_DATA_2; footprint (none) -> Custom_TestPoint:TestPoint_LoopPostPad
- TP2: value (none) -> GND; footprint (none) -> Custom_TestPoint:TestPoint_LoopPostPad
- TP20: value (none) -> SLIDE_DATA_3; footprint (none) -> Custom_TestPoint:TestPoint_LoopPostPad
- TP21: value (none) -> ROT_DATA_0; footprint (none) -> Custom_TestPoint:TestPoint_LoopPostPad
- TP22: value (none) -> ROT_DATA_1; footprint (none) -> Custom_TestPoint:TestPoint_LoopPostPad
- TP23: value (none) -> ROT_DATA_2; footprint (none) -> Custom_TestPoint:TestPoint_LoopPostPad
- TP24: value (none) -> ROT_DATA_3; footprint (none) -> Custom_TestPoint:TestPoint_LoopPostPad
- TP3: value (none) -> DATA_0; footprint (none) -> Custom_TestPoint:TestPoint_LoopPostPad
- TP4: value (none) -> DATA_1; footprint (none) -> Custom_TestPoint:TestPoint_LoopPostPad
- TP5: value (none) -> DATA_2; footprint (none) -> Custom_TestPoint:TestPoint_LoopPostPad
- TP6: value (none) -> DATA_3; footprint (none) -> Custom_TestPoint:TestPoint_LoopPostPad
- U1: value (none) -> Hexadecimal; footprint (none) -> Display_7Segment:HDSP-A151
- U2: value (none) -> Decimal; footprint (none) -> Display_7Segment:DA56-11SURKWA
Connections:
- net DIG1: now reaches Q1.3 (D), U1.1 (CC), U1.6 (CC)
- net DIG3: now reaches Q3.3 (D), U2.13 (DIG2_CC)
- net DIG2: now reaches Q2.3 (D), U2.14 (DIG1_CC)
Other:
- moved on the sheet: Q1, Q2, Q3
